File: stdc14-to-100mil-breakout/stdc14-to-100mil-breakout.kicad_sch (KiCad schematic)
At the start: 5 parts, among them J1 STDC14_MaleReceptacle_TargetS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, J2 PinHeader_1x07_P2.54mm_Vertic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, J3 PinHeader_1x07_P2.54mm_Vertic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, J4 PinHeader_1x08_P2.54mm_Vertic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, J5 PinHeader_1x02_P2.54mm_Vertic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

Commit message: Add part numbers for stdc connector
Parts:
- J1: distr1 (none) -> Digikey; distr1# (none) -> 1175-1736-ND; distr2 (none) -> Digikey; distr2# (none) -> SAM12420-ND; manf1 (none) -> CNC Tech; manf1# (none) -> 3221-14-0100-00; manf2 (none) -> Samtec Inc.; manf2# (none) -> FTSH-107-01-S-D-K
